Commit message: omniwheel desc.

File: models/omnidirectional/robot.urdf (robot description, URDF)
Before this commit: robot onshape, 65 links, 64 joints
Joints:
- removed joint wheel1_speed
- removed joint wheel2_speed
- removed joint wheel3_speed
- added joint wheel_1: type revolute, parent body, child wheel, origin xyz=0.069282032302755147679 -0.039999999999999986955 0.012999999999999999403 rpy=-1.570796326794896558 -0 1.0471975511965980754, axis 0 0 1, limit effort=1 velocity=20
- added joint wheel_2: type revolute, parent body, child wheel_3, origin xyz=-6.5919492087118669588e-17 0.080000000000000182077 0.013000000000000034098 rpy=1.570796326794896558 -0 6.1062266354383451951e-16, axis 0 0 1, limit effort=1 velocity=20
- added joint wheel_3: type revolute, parent body, child wheel_2, origin xyz=-0.069282032302755092168 -0.040000000000000063283 0.012999999999999999403 rpy=1.570796326794896558 -0 2.0943951023931961508, axis 0 0 1, limit effort=1 velocity=20

Commit message: Omni joint names

File: models/omnidirectional/robot.urdf (robot description, URDF)
Before this commit: robot onshape, 65 links, 64 joints
Joints:
- removed joint wheel_1
- removed joint wheel_2
- removed joint wheel_3
- added joint wheel1: type revolute, parent body, child wheel, origin xyz=0.069282032302755147679 -0.039999999999999986955 0.012999999999999999403 rpy=-1.570796326794896558 -0 1.0471975511965980754, axis 0 0 1, limit effort=1 velocity=20
- added joint wheel2: type revolute, parent body, child wheel_3, origin xyz=-6.5919492087118669588e-17 0.080000000000000182077 0.013000000000000034098 rpy=1.570796326794896558 -0 6.1062266354383451951e-16, axis 0 0 1, limit effort=1 velocity=20
- added joint wheel3: type revolute, parent body, child wheel_2, origin xyz=-0.069282032302755092168 -0.040000000000000063283 0.012999999999999999403 rpy=1.570796326794896558 -0 2.0943951023931961508, axis 0 0 1, limit effort=1 velocity=20
