Commit message: Orbita robot

File: models/orbita/robot.urdf (robot description, URDF)
Before this commit: robot onshape, 13 links, 12 joints
Links:
- removed link closing_br2_1
- removed link closing_br2_2
- removed link closing_br3_1
- removed link closing_br3_2
- added link closing_ring2_br2_1, mass 1e-9
- added link closing_ring2_br2_2, mass 1e-9
- added link closing_ring3_br2_1, mass 1e-9
- added link closing_ring3_br2_2, mass 1e-9
- link ring2: mass 1.2478922652256831949 -> 1.2478922652256829728
Joints:
- removed joint closing_br2_1_frame
- removed joint closing_br2_2_frame
- removed joint closing_br3_1_frame
- removed joint closing_br3_2_frame
- added joint closing_ring2_br2_1_frame: type fixed, parent platform, child closing_ring2_br2_1, origin xyz=-0.070148057706539423961 3.0531133177191804862e-16 -0.12149999999999989975 rpy=3.141592653589788231 -1.0471975511965971872 -3.1415926535897917837, axis 0 0 0
- added joint closing_ring2_br2_2_frame: type fixed, parent branch, child closing_ring2_br2_2, origin xyz=0.080999999999999988676 2.7755575615628913511e-17 -0.099000000000000032419 rpy=-1.5707963267948970021 -5.488882269908094325e-17 -1.570796326794896558, axis 0 0 0
- added joint closing_ring3_br2_1_frame: type fixed, parent platform, child closing_ring3_br2_1, origin xyz=0.070148057706539437839 3.0531133177191804862e-16 -0.12149999999999985811 rpy=-3.141592653589788231 -1.0471975511965980754 -1.4837675049255949395e-15, axis 0 0 0
- added joint closing_ring3_br2_2_frame: type fixed, parent branch_2, child closing_ring3_br2_2, origin xyz=0.080999999999999988676 -2.7755575615628913511e-17 -0.099000000000000004663 rpy=1.5707963267948970021 6.4413030524365536505e-17 1.570796326794896558, axis 0 0 0

Commit message: Adding base frame in orbita

File: models/orbita/robot.urdf (robot description, URDF)
Before this commit: robot onshape, 13 links, 12 joints
Links:
- added link bottom, mass 1.6751498268076565612; collision mesh filename=package:///bottom.stl; visual mesh filename=package:///bottom.stl
- link base: mass 1.6751498268076565612 -> 1e-9; geometry 
Joints:
- added joint base_frame: type fixed, parent bottom, child base, origin xyz=3.3702370129303403613e-19 -1.530808498935084399e-19 0.10200000000000000733 rpy=3.117578297433438655e-27 -3.6603146002254947771e-27 -2.4671464441025585051e-27, axis 0 0 0
- joint closing_ring2_br2_2_frame: origin xyz=0.080999999999999988676 2.7755575615628913511e-17 -0.099000000000000032419 rpy=-1.5707963267948970021 -5.488882269908094325e-17 -1.570796326794896558 -> xyz=0.080999999999999988676 2.7755575615628913511e-17 -0.099000000000000004663 rpy=-1.57079632679489678 -5.5511151231257827021e-17 -1.570796326794896558
- joint closing_ring3_br2_1_frame: origin xyz=0.070148057706539437839 3.0531133177191804862e-16 -0.12149999999999985811 rpy=-3.141592653589788231 -1.0471975511965980754 -1.4837675049255949395e-15 -> xyz=0.070148057706539451717 3.0531133177191804862e-16 -0.12149999999999985811 rpy=-3.141592653589788231 -1.0471975511965980754 -1.4837675049255951367e-15
- joint closing_ring3_br2_2_frame: origin xyz=0.080999999999999988676 -2.7755575615628913511e-17 -0.099000000000000004663 rpy=1.5707963267948970021 6.4413030524365536505e-17 1.570796326794896558 -> xyz=0.080999999999999974798 0 -0.099000000000000004663 rpy=1.5707963267948970021 5.5511151231257839347e-17 1.570796326794896558
- joint effector_frame: origin xyz=-3.3702370129283359497e-19 0.012000000000000066169 -0.080999999999999905409 rpy=1.5707963267948936714 -1.2286129093570810081e-27 3.141592653589793116 -> xyz=-3.3702370129283359497e-19 0.012000000000000066169 -0.080999999999999905409 rpy=1.5707963267948936714 -1.2283261469517751369e-27 3.141592653589793116
- joint ring1: parent base -> bottom
- joint ring1_br1: origin xyz=0.070003571337468123437 -2.0497195342395766699e-17 -0.051169047558312585888 rpy=-0.78539816339743695472 1.6076990612689687564e-14 -1.5707963267948796826 -> xyz=0.070003571337468123437 -6.6194075345813099437e-18 -0.051169047558312585888 rpy=-0.78539816339743695472 1.6098233857064223944e-14 -1.5707963267948796826
- joint ring1_br2: origin xyz=0.081000000000003208322 -1.0824674490095276269e-15 -0.099000000000000157319 rpy=-1.5707963267948970021 0.78539816339745016638 -1.570796326794896558 -> xyz=0.081000000000003236078 -1.0269562977782697999e-15 -0.099000000000000157319 rpy=-1.5707963267948970021 0.78539816339745016638 -1.570796326794896558
- joint ring2: parent base -> bottom
- joint ring2_br1: origin xyz=-0.035001785668734054779 0.060624871133883498353 -0.099169047558312600765 rpy=-0.78539816339744594753 -1.5947199972316488546e-14 0.5235987755982836056 -> xyz=-0.035001785668734061718 0.060624871133883498353 -0.099169047558312600765 rpy=-0.78539816339744594753 -1.5931700114609247704e-14 0.5235987755982836056
- joint ring3: parent base -> bottom
- joint ring3_br1: origin xyz=-0.03500178566873398539 -0.060624871133883539986 -0.075169047558312648838 rpy=-0.78539816339743317997 6.8726209472379501374e-15 2.6179938779915028491 -> xyz=-0.03500178566873398539 -0.060624871133883539986 -0.075169047558312648838 rpy=-0.78539816339743317997 6.8833827526758766762e-15 2.6179938779915028491
