Commit message: Planar 2DoF + examples

File: models/planar-2dof/robot.urdf (robot description, URDF)
Before this commit: robot onshape, 8 links, 7 joints
Links:
- link branch2: mass 0.11287599307230633539 -> 0.11287599307230634926
- link branch2_2: mass 0.11287599307230633539 -> 0.11287599307230634926
Joints:
- joint closing_effector_1_frame: origin xyz=0.064999999999999988343 0.075993420767853286923 0.004999999999999997502 rpy=0 -0 5.5511151231257827021e-17 -> xyz=0.065000000000000016098 0.075993420767853314679 0.0050000000000000027062 rpy=0 -4.8148248609680896326e-34 -1.3877787807814456755e-17
- joint closing_effector_2_frame: origin xyz=0.065000000000000029976 0.075993420767853286923 0.0050000000000000009714 rpy=3.141592653589793116 6.1629758220391547298e-33 1.570796326794896558 -> xyz=0.06500000000000000222 0.075993420767853286923 0.0050000000000000044409 rpy=3.141592653589793116 -0 1.570796326794896558
- joint effector_frame: origin xyz=0.065000000000000029976 0.075993420767853286923 -0.010000000000000005412 rpy=3.141592653589793116 -1.7252291750463170016e-17 -5.551115123125917055e-17 -> xyz=0.06500000000000000222 0.075993420767853342435 -0.009999999999999995004 rpy=-3.1415926535897922278 -1.9150136985426451064e-16 2.7755575615628106161e-17
- joint motor1: origin xyz=0.014999999999999999445 -0.060000000000000011657 0.045000000000000012212 rpy=-1.570796326794896558 0.22112146340132790567 1.570796326794896558 -> xyz=0.014999999999999995975 -0.059999999999999970024 0.044999999999999991396 rpy=-1.570796326794896336 0.54685095069594424899 1.570796326794896558
- joint motor2: origin xyz=0.015000000000000006384 0.05999999999999999778 0.045000000000000005274 rpy=1.570796326794896558 0.22112146340130267586 -1.570796326794896336 -> xyz=0.014999999999999999445 0.059999999999999983902 0.044999999999999991396 rpy=1.570796326794896558 0.54685095069594436001 -1.570796326794896336
- joint passive1: origin xyz=-0.065000000000000224265 -0.10677078252031298178 -5.0306980803327405738e-17 rpy=3.141592653589793116 -2.3755581631045393401e-16 0.6420904266682142536 -> xyz=-0.065000000000000210387 -0.1067707825203129679 0 rpy=3.141592653589793116 -2.3043122745956649559e-16 -0.61093427862802440753
- joint passive2: origin xyz=-0.065000000000000224265 0.10677078252031305117 -0.0099999999999999967387 rpy=9.1577368045060010207e-17 -1.1716466983231724797e-16 -0.64209042666824067691 -> xyz=-0.065000000000000224265 0.10677078252031299566 -0.010000000000000007147 rpy=-4.1402727141222208915e-16 -5.0706060260327139801e-17 0.61093427862801419348
