Commit message: Megabot update

File: models/megabot/robot.urdf (robot description, URDF)
Before this commit: robot megabot, 82 links, 81 joints
Links:
- link center: mass 139.99113879410856498 -> 139.99113879410870709
- link cylinder_f: mass 2.7501984867936557499 -> 2.7501984867936553059
- link cylinder_f_10: mass 2.7501984867936557499 -> 2.7501984867936553059
- link cylinder_f_11: mass 2.7501984867936557499 -> 2.7501984867936553059
- link cylinder_f_12: mass 2.7501984867936557499 -> 2.7501984867936553059
- link cylinder_f_2: mass 2.7501984867936557499 -> 2.7501984867936553059
- link cylinder_f_3: mass 2.7501984867936557499 -> 2.7501984867936553059
- link cylinder_f_4: mass 2.7501984867936557499 -> 2.7501984867936553059
- link cylinder_f_5: mass 2.7501984867936557499 -> 2.7501984867936553059
- link cylinder_f_6: mass 2.7501984867936557499 -> 2.7501984867936553059
- link cylinder_f_7: mass 2.7501984867936557499 -> 2.7501984867936553059
- link cylinder_f_8: mass 2.7501984867936557499 -> 2.7501984867936553059
- link cylinder_f_9: mass 2.7501984867936557499 -> 2.7501984867936553059
- link cylinder_support: mass 3.4500000005941271475 -> 3.4500000005941280357
- link cylinder_support_2: mass 3.4500000005941271475 -> 3.4500000005941280357
- link cylinder_support_3: mass 3.4500000005941271475 -> 3.4500000005941280357
- link cylinder_support_4: mass 3.4500000005941271475 -> 3.4500000005941280357
- link femur: mass 3.5999999984857389279 -> 3.5999999984857375956
- link femur_2: mass 3.5999999984857389279 -> 3.5999999984857375956
- link femur_3: mass 3.5999999984857389279 -> 3.5999999984857375956
- link femur_4: mass 3.5999999984857389279 -> 3.5999999984857375956
- link hip: mass 3.5999999924476488999 -> 3.5999999924476484559
- link hip_2: mass 3.5999999924476488999 -> 3.5999999924476484559
- link hip_3: mass 3.5999999924476488999 -> 3.5999999924476484559
- link hip_4: mass 3.5999999924476488999 -> 3.5999999924476484559
- link tibia: mass 3.999999995260936636 -> 3.999999995260936192
- link tibia_2: mass 3.999999995260936636 -> 3.999999995260936192
- link tibia_3: mass 3.999999995260936636 -> 3.999999995260936192
- link tibia_4: mass 3.999999995260936636 -> 3.999999995260936192
Joints:
- joint l1_c1: origin xyz=0.54016194822255925168 8.8817841970012523234e-16 1.7017248921313462451e-16 rpy=-1.3601114862349504746e-17 1.570796326794896336 0 -> xyz=0.45949999999998797362 -1.1102230246251565404e-16 6.1825161828937341108e-16 rpy=1.5839373449339953594e-15 1.5707963267948945596 0
- joint l1_c2: origin xyz=0.50159604710364502633 1.6653345369377348106e-15 -2.553512956637860043e-15 rpy=-1.4830109546207050645e-15 1.5707963267948930053 0 -> xyz=0.45949999999999657785 4.4408920985006261617e-16 -4.0141501234103316165e-15 rpy=-9.0093448943835609015e-16 1.5707963267948890085 0
- joint l1_c3: origin xyz=0.55992619355683259652 1.5543122344752191566e-15 6.7168492989821970696e-15 rpy=3.1415926535897864547 -1.570796326794891673 0 -> xyz=0.45949999999999446842 2.664535259100375697e-15 -2.1649348980190552538e-15 rpy=-3.1415926535897926719 -1.570796326794896336 0
- joint l1_cl1_1_frame: origin xyz=0 0 -0.0095000000000000639488 rpy=-1.570796326794896558 -1.570796326794896558 0 -> xyz=3.9443045261050590271e-31 -5.5511151231257827021e-17 -0.0094999999999999529265 rpy=-1.570796326794896558 -1.570796326794896558 0
- joint l1_cl1_2_frame: origin xyz=0.27500000000000013323 -5.5511151231257827021e-17 0.030000000000000002359 rpy=-1.570796326794896336 1.3210496169531149881e-16 -3.141592653589793116 -> xyz=0.27499999999999968914 -3.8163916471489756077e-17 0.030000000000000005829 rpy=-1.570796326794896336 1.3210496169531085786e-16 -3.141592653589793116
- joint l1_cl2_1_frame: origin xyz=-4.4408920985006261617e-16 1.1102230246251565404e-16 -0.0094999999999998419042 rpy=-1.570796326794896558 -1.5707963267948958919 0 -> xyz=2.185751579730776939e-16 0 -0.0094999999999999529265 rpy=-1.57079632679489678 -1.5707963267948952257 0
- joint l1_cl2_2_frame: origin xyz=-0.012999999999999789502 0.38400000000000000799 0.019999999999999795719 rpy=1.57079632679489678 7.2637879135570270462e-17 -6.7181087869012247853e-17 -> xyz=-0.012999999999999900524 0.38400000000000011902 0.019999999999999868577 rpy=1.57079632679489678 -3.1065260723641943717e-16 -7.2676014924345448372e-17
- joint l1_cl3_1_frame: origin xyz=1.1102230246251565404e-16 0 -0.0094999999999996198596 rpy=1.57079632679489678 1.570796326794896336 0 -> xyz=1.7347234759768070944e-17 2.2204460492503130808e-16 -0.0095000000000002859935 rpy=1.57079632679489678 1.570796326794896558 0
- joint l1_cl3_2_frame: origin xyz=-2.2204460492503130808e-16 -0.50500000000000011546 0.020000000000000184297 rpy=-1.570796326794896558 5.9381623995301617414e-16 3.141592653589793116 -> xyz=2.2204460492503130808e-16 -0.50500000000000033751 0.020000000000000052458 rpy=-1.570796326794896558 5.6756690386264740081e-16 3.141592653589793116
- joint l1_cl4_1_frame: origin xyz=0 0.58999999999999996891 0.019999999999999573674 rpy=1.5707963267948936714 -3.6993336504632930902e-17 -3.141592653589793116 -> xyz=2.2204460492503130808e-16 0.59000000000000007994 0.020000000000000097561 rpy=1.5707963267948961139 -2.5998066656079383138e-17 -3.141592653589793116
- joint l1_cl4_2_frame: origin xyz=-0.44999999999999995559 0 -0.020000000000000184297 rpy=-1.570796326794896558 6.5422720734645307412e-18 -3.141592653589793116 -> xyz=-0.44999999999999973355 1.1102230246251565404e-16 -0.01999999999999997613 rpy=-1.570796326794896558 3.3141074150295935238e-16 -3.141592653589793116
- joint l1_r1: origin xyz=-0.44000000000000016875 -0.33500000000000024203 1.0755285551056207683e-16 rpy=3.1415926535897922278 -2.3595482621880709577e-16 -1.2888338553123910302 -> xyz=-0.44000000000000022427 -0.33500000000000051958 1.0755285551056216311e-16 rpy=3.1415926535897926719 1.5635084904658178429e-16 -1.433149400124039019
- joint l1_r2: origin xyz=-0.50000000000000011102 -1.0250000000000001332 0.030000000000000102973 rpy=3.141592653589793116 -3.0599760784490747333e-18 0.71499248882173183084 -> xyz=-0.49999999999999811262 -1.0249999999999999112 0.030000000000000102973 rpy=3.141592653589793116 -3.0599681271326078913e-18 1.0975074011255603335
- joint l1_r3: origin xyz=0.12500000000000022204 -0.019999999999999906741 -0.040000000000000007772 rpy=-1.570796326794896558 0.35430516897438335544 8.333430058132758542e-15 -> xyz=0.12499999999999977796 -0.019999999999999826944 -0.039999999999999993894 rpy=-1.5707963267948956698 0.46670348839401742946 -4.1843661536946179153e-16
- joint l1_r4: origin xyz=-1.1102230246251565404e-16 0.48999999999999999112 -2.2204460492503130808e-16 rpy=3.1415926535897900074 2.7294237846170472709e-15 -0.35430516897438252277 -> xyz=3.3306690738754696213e-16 0.4899999999999998801 -1.9949319973733281586e-17 rpy=3.141592653589793116 9.8174925928936230861e-16 -0.41532921468036260171
- joint l1_r5: origin xyz=-0.75 -1.1102230246251565404e-16 -0.040000000000000146549 rpy=-5.6175769265896188431e-16 1.3875289317899453937e-15 3.141592653589793116 -> xyz=-0.74999999999999977796 0 -0.040000000000000153488 rpy=-1.3519093026149155761e-15 1.7849770799465899747e-15 2.8740211174390379867
- joint l1_r6: origin xyz=-0.40999999999999992006 1.6653345369377348106e-16 -0.094999999999999987232 rpy=1.570796326794896558 0.65724109672367558854 -6.6514940932233617718e-15 -> xyz=-0.41000000000000014211 1.2836953722228372499e-16 -0.095000000000000014988 rpy=1.57079632679489678 0.67750901888019166019 1.6143341020285157788e-15
- joint l1_r7: origin xyz=-0.12499999999999822364 -0.020000000000001849632 -0.040000000000000007772 rpy=-1.570796326794896558 0.67784852797306960337 -1.2527273977519951284e-15 -> xyz=-0.12500000000000066613 -0.020000000000001065537 -0.040000000000004920508 rpy=-1.5707963267949032193 0.79185786258827683959 -1.7629992927556572186e-14
- joint l1_r8: origin xyz=2.2204460492503130808e-16 0.39249999999999996003 0.020000000000001461054 rpy=6.6758930342687408726e-15 1.8103960944874226249e-14 -3.1275650633842229098 -> xyz=-9.9920072216264088638e-16 0.3925000000000082867 0.020000000000004944378 rpy=2.2502960553273176995e-14 3.8695720785859771458e-14 -3.0319894979551293979
- joint l2_c1: origin xyz=0.54016194822256369257 -3.6082248300317587564e-16 9.9643341442874709379e-17 rpy=1.7558505235703240888e-16 1.5707963267948950037 0 -> xyz=0.45950000080081426779 5.5511151231257827021e-17 7.9271560598040820885e-17 rpy=1.7200196442759473774e-16 1.5707963267948950037 0
- joint l2_c2: origin xyz=0.50159604710360994329 0 1.4988010832439613296e-15 rpy=1.072854554705450715e-16 1.5707963267948927832 0 -> xyz=0.4595000000000002971 1.7763568394002504647e-15 2.3869795029440865619e-15 rpy=3.4013390378763887518e-16 1.5707963267948954478 0
- joint l2_c3: origin xyz=0.55992619355683270754 -2.4424906541753443889e-15 5.1070259132757200859e-15 rpy=3.1415926535897789051 -1.5707963267948827912 0 -> xyz=0.45950000000000035261 -5.5511151231257827021e-15 1.0824674490095276269e-14 rpy=3.1415926535897802374 -1.5707963267948861219 0
- joint l2_cl1_1_frame: origin xyz=9.8607613152626475676e-32 0 -0.0095000000000000639488 rpy=-1.5707963267948970021 -1.5707963267948954478 0 -> xyz=9.8607613152626475676e-32 0 -0.00950000000000011946 rpy=-1.5707963267948970021 -1.5707963267948954478 0
- joint l2_cl1_2_frame: origin xyz=0.2750000000000000222 5.5511151231257827021e-17 0.02999999999999999889 rpy=-1.570796326794896336 5.8999261890123604462e-17 -3.1415926535897926719 -> xyz=0.27500000000000013323 -5.5511151231257827021e-17 0.02999999999999999889 rpy=-1.570796326794896336 5.8999261890123592136e-17 -3.1415926535897926719
- joint l2_cl2_1_frame: origin xyz=5.5511151231257827021e-17 -1.1102230246251565404e-16 -0.0094999999999999962946 rpy=-1.570796326794896558 -1.5707963267948930053 0 -> xyz=1.1102230246251565404e-16 0 -0.0094999999999999945599 rpy=-1.570796326794896336 -1.5707963267948927832 0
- joint l2_cl2_2_frame: origin xyz=-0.013000000000000011546 0.38400000000000000799 0.020000000000000073275 rpy=1.570796326794896558 -2.9099399159039228985e-16 -7.2338255418286372255e-17 -> xyz=-0.012999999999999706235 0.3840000000000000635 0.019999999999999962252 rpy=1.570796326794896558 1.4889190345132270871e-16 3.4804450275470782491e-17
- joint l2_cl3_1_frame: origin xyz=1.6653345369377348106e-16 0 -0.0095000000000000639488 rpy=1.570796326794896558 1.5707963267948956698 0 -> xyz=5.5511151231257827021e-17 0 -0.0094999999999998419042 rpy=1.570796326794896558 1.5707963267948956698 0
- joint l2_cl3_2_frame: origin xyz=0 -0.50500000000000000444 0.020000000000000017764 rpy=-1.570796326794896558 -8.5901255498107134466e-16 -3.141592653589793116 -> xyz=2.2204460492503130808e-16 -0.50499999999999989342 0.020000000000000239808 rpy=-1.57079632679489678 -1.1929415864978866461e-15 3.141592653589793116
- joint l2_cl4_1_frame: origin xyz=0 0.58999999999999996891 0.020000000000000184297 rpy=1.5707963267948941155 -6.8893610029579801103e-15 -3.141592653589793116 -> xyz=-5.5511151231257827021e-17 0.5899999999999994138 0.019999999999999712452 rpy=1.5707963267948938935 -7.2175292787070834916e-15 -3.141592653589793116
- joint l2_cl4_2_frame: origin xyz=-0.44999999999999990008 0 -0.01999999999999985123 rpy=-1.570796326794896558 2.0671484703801979509e-17 3.141592653589793116 -> xyz=-0.44999999999999984457 2.2204460492503130808e-16 -0.020000000000000073275 rpy=-1.570796326794896558 -2.4707137350212771429e-16 3.141592653589793116
- joint l2_r1: origin xyz=0.18999999999999972466 -0.08499999999999972855 1.0755285551056199055e-16 rpy=3.141592653589793116 -1.6993414331267333812e-16 -2.8596301821072906968 -> xyz=0.18999999999999978018 -0.084999999999999686917 1.0755285551056200288e-16 rpy=3.141592653589793116 -7.1582305289484675573e-17 -2.9958563448520303396
- joint l2_r2: origin xyz=-0.50000000000000011102 -0.024999999999999852202 0.030000000000000096034 rpy=3.141592653589793116 -1.1535304933115970508e-16 -0.85580383797315651151 -> xyz=-0.50000000000000022204 -0.024999999999999900774 0.030000000000000106443 rpy=3.141592653589793116 -1.153529978888650079e-16 -0.47328893068798266741
- joint l2_r3: origin xyz=0.12500000000000011102 -0.02000000000000035083 -0.040000000000000028588 rpy=-1.570796326794896336 0.35430516897447805746 -2.2175415972529100751e-15 -> xyz=0.12499999999999977796 -0.019999999999999934497 -0.040000000000000042466 rpy=-1.5707963267948978903 0.46670348839402453489 -6.6556317978518277341e-15
- joint l2_r4: origin xyz=1.6653345369377348106e-16 0.48999999999999965805 -4.4408920985006261617e-16 rpy=3.141592653589793116 -3.4782139178269834916e-15 -0.35430516897447428271 -> xyz=-6.9388939039072283776e-16 0.48999999999999993561 6.6613381477509392425e-16 rpy=3.1415926535897926719 -1.0377520731080190909e-14 -0.41532921468034922352
- joint l2_r5: origin xyz=-0.75 -1.1102230246251565404e-16 -0.039999999999999980016 rpy=-9.4612926646945399132e-16 1.9371594980863719444e-16 -3.141592653589793116 -> xyz=-0.74999999999999988898 1.1102230246251565404e-16 -0.040000000000000091038 rpy=2.540715062519631097e-16 -2.943161147134564992e-15 2.864108120675692426
- joint l2_r6: origin xyz=-0.40999999999999980904 7.2164496600635175128e-16 -0.095000000000000028866 rpy=1.570796326794896558 0.65724109672367858614 -5.1466463596763776877e-15 -> xyz=-0.409999999999999587 -4.9960036108132044319e-16 -0.094999999999999723554 rpy=1.5707963267948961139 0.67750901888017123209 1.6649055331051427788e-15
- joint l2_r7: origin xyz=-0.1249999999999990008 -0.019999999999999074074 -0.040000000000000000833 rpy=-1.570796326794896558 0.67784852797311845318 6.530241321319161551e-15 -> xyz=-0.1249999999999990008 -0.020000000000000600631 -0.039999999999999875933 rpy=-1.5707963267948978903 0.79185786258829393702 1.7746994413076171452e-15
- joint l2_r8: origin xyz=2.2204460492503130808e-16 0.39249999999999984901 0.01999999999999985123 rpy=6.0491518543493472829e-15 3.6588336647256622468e-15 -3.1275650633842677628 -> xyz=1.9984014443252817728e-15 0.3924999999999977951 0.020000000000001932898 rpy=1.6800334858317061208e-14 2.9059497397685848373e-14 -3.0259156815526302431
- joint l3_c1: origin xyz=0.54016194822258023489 3.1086244689504383132e-15 -9.140831766129502433e-16 rpy=-1.8325883609705074827e-16 1.5707963267948930053 0 -> xyz=0.45949999999999835421 5.5511151231257827021e-16 -5.3489951134560793381e-16 rpy=-1.0364157664800512015e-16 1.5707963267948930053 0
- joint l3_c2: origin xyz=0.5015960471036677859 -4.4408920985006261617e-16 2.2204460492503130808e-16 rpy=-6.354613258499769017e-17 1.5707963267948921171 0 -> xyz=0.45950000000000540412 9.4924068605450884206e-15 -9.0483176506950258045e-15 rpy=-2.8571979860306309276e-16 1.5707963267948910069 0
- joint l3_c3: origin xyz=0.55992619355682637927 -3.5527136788005009294e-15 -2.2204460492503130808e-15 rpy=-3.141592653589793116 -1.570796326794896336 0 -> xyz=0.45949999999999446842 -1.5543122344752191566e-15 9.9920072216264088638e-16 rpy=3.1415926535897829019 -1.5707963267948807928 0
- joint l3_cl1_1_frame: origin xyz=0 2.7755575615628913511e-17 -0.0095000000000000084377 rpy=-1.570796326794896558 -1.570796326794896558 0 -> xyz=3.9443045261050590271e-31 0 -0.0094999999999998974154 rpy=-1.570796326794896558 -1.570796326794896558 0
- joint l3_cl1_2_frame: origin xyz=0.27499999999999980016 0 0.02999999999999999889 rpy=-1.570796326794896558 -4.4969093478228596159e-29 3.1415926535897922278 -> xyz=0.27499999999999985567 0 0.02999999999999999889 rpy=-1.570796326794896558 -4.4993958156375995493e-29 3.1415926535897926719
- joint l3_cl2_1_frame: origin xyz=-5.5511151231257827021e-17 0 -0.0094999999999999668043 rpy=-1.5707963267948972241 -1.570796326794896336 0 -> xyz=0 -5.5511151231257827021e-17 -0.009499999999999987621 rpy=-1.5707963267948974462 -1.5707963267948961139 0
- joint l3_cl2_2_frame: origin xyz=-0.013000000000000067057 0.3840000000000000635 0.020000000000000017764 rpy=1.570796326794896558 -5.2424180237022428121e-16 -6.8688372249162086865e-17 -> xyz=-0.012999999999999886646 0.38400000000000011902 0.019999999999999962252 rpy=1.5707963267948985564 -4.1117207255037771762e-15 -1.2965582971512668008e-16
- joint l3_cl3_1_frame: origin xyz=-1.1102230246251565404e-16 0 -0.0094999999999997308819 rpy=1.57079632679489678 1.570796326794896336 0 -> xyz=-1.1102230246251565404e-16 0 -0.0094999999999999529265 rpy=1.57079632679489678 1.5707963267948874542 0
- joint l3_cl3_2_frame: origin xyz=0 -0.50499999999999989342 0.020000000000000073275 rpy=-1.570796326794896558 3.5164344829539952788e-16 3.1415926535897926719 -> xyz=0 -0.50500000000000011546 0.020000000000000073275 rpy=-1.570796326794896558 -5.2716164429158478364e-17 -3.141592653589793116
- joint l3_cl4_1_frame: origin xyz=-1.6653345369377348106e-16 0.59000000000000007994 0.019999999999999962252 rpy=1.570796326794896558 -9.0419128252829653613e-17 3.141592653589793116 -> xyz=8.3266726846886740532e-17 0.58999999999999996891 0.019999999999999962252 rpy=1.5707963267949054398 9.6515610006004477964e-15 3.141592653589793116
- joint l3_cl4_2_frame: origin xyz=-0.45000000000000012212 -1.1102230246251565404e-16 -0.019999999999999906741 rpy=-1.570796326794896558 -7.1621134632402218173e-17 3.141592653589793116 -> xyz=-0.44999999999999990008 0 -0.019999999999999962252 rpy=-1.570796326794896558 2.2761969218518991462e-16 3.141592653589793116
- joint l3_r1: origin xyz=0.44000000000000055733 -0.71499999999999974687 1.0755285551056202753e-16 rpy=-3.1415926535897904515 3.2403040233095439527e-24 1.8527587982774034181 -> xyz=0.43999999999999966915 -0.71499999999999852562 1.0755285551057660913e-16 rpy=-3.1415926535897904515 1.1842700142122408505e-24 1.7165326330347507877
- joint l3_r2: origin xyz=0.49999999999999994449 -0.024999999999999918121 0.030000000000000102973 rpy=-3.1415926535897922278 -8.7006547959070078248e-16 -2.4266001647680677245 -> xyz=0.5 -0.024999999999999918121 0.030000000000000102973 rpy=-3.1415926535897926719 -7.5808492435147575872e-16 -2.0440852524641424104
- joint l3_r3: origin xyz=0.12499999999999980571 -0.019999999999999962252 -0.04000000000000001471 rpy=-1.57079632679489678 0.35430516897432023926 6.1122737486658637803e-15 -> xyz=0.12499999999999167333 -0.01999999999999840794 -0.040000000000000097977 rpy=-1.5707963267948958919 0.46670348839395431328 -8.9960860717502477891e-15
- joint l3_r4: origin xyz=-2.7755575615628913511e-17 0.49000000000000004663 -5.5511151231257827021e-17 rpy=3.1415926535897873428 2.9877259684137084701e-15 -0.35430516897432418055 -> xyz=4.1633363423443370266e-16 0.48999999999999943601 1.6098233857064769836e-15 rpy=-3.1415926535897895633 -1.1450887451527557207e-14 -0.41532921468024797118
- joint l3_r5: origin xyz=-0.75000000000000022204 0 -0.03999999999999970246 rpy=-1.1255613980499141844e-15 -3.2685853399614706325e-15 -3.141592653589793116 -> xyz=-0.75 0 -0.040000000000000146549 rpy=-1.2697226730609879444e-15 1.6397443508591157754e-15 2.8709603175061224611
- joint l3_r6: origin xyz=-0.4100000000000000866 4.9960036108132044319e-16 -0.095000000000000056621 rpy=1.5707963267948994446 0.65724109672367359014 1.8096855595557680072e-15 -> xyz=-0.40999999999999930944 -1.6653345369377348106e-15 -0.095000000000000750511 rpy=1.5707963267948974462 0.67750901888020520492 -4.8652669090637057603e-15
- joint l3_r7: origin xyz=-0.12500000000000011102 -0.019999999999999795719 -0.039999999999999986955 rpy=-1.57079632679489678 0.67784852797300643168 -3.8844866652341196646e-15 -> xyz=-0.12499999999999988898 -0.020000000000000905942 -0.039999999999999431843 rpy=-1.57079632679489678 0.79185786258829671258 -1.035821479701865864e-14
- joint l3_r8: origin xyz=-5.5511151231257827021e-17 0.39250000000000023759 0.019999999999999962252 rpy=-1.4752362061541671842e-15 -1.1273800577279551433e-15 -3.1275650633841585169 -> xyz=1.7763568394002504647e-15 0.39249999999999962697 0.020000000000000128786 rpy=1.3451873289489358511e-14 1.1341460953105552235e-14 -3.0301163114049525227
- joint l4_c1: origin xyz=0.54016194822257568298 -1.1102230246251565404e-16 3.2215294379649110445e-16 rpy=1.9525057998941007146e-16 1.5707963267948952257 0 -> xyz=0.45949999999999974198 -9.9920072216264088638e-16 7.9164734028173481031e-17 rpy=2.7892200453038867559e-16 1.5707963267948952257 0
- joint l4_c2: origin xyz=0.5015960471036094992 -1.1102230246251565404e-15 -1.9984014443252817728e-15 rpy=-1.4206229417985893165e-15 1.5707963267948938935 0 -> xyz=0.45949999999999890932 -5.5511151231257827021e-16 -8.8817841970012523234e-16 rpy=1.7957032038766200501e-15 1.5707963267948890085 0
- joint l4_c3: origin xyz=0.55992619355684736249 -3.7747582837255322374e-15 4.8294701571194309508e-15 rpy=3.1415926535897864547 -1.5707963267948921171 0 -> xyz=0.45949999999999957545 4.4408920985006261617e-16 3.3306690738754696213e-16 rpy=-3.1415926535897926719 -1.5707963267948958919 0
- joint l4_cl1_1_frame: origin xyz=0 0 -0.0094999999999999668043 rpy=-1.570796326794896558 -1.570796326794896336 0 -> xyz=9.8607613152626475676e-32 -1.1102230246251565404e-16 -0.0095000000000000361933 rpy=-1.570796326794896558 -1.570796326794896336 0
- joint l4_cl1_2_frame: origin xyz=0.2750000000000000222 1.1102230246251565404e-16 0.029999999999999991951 rpy=-1.5707963267948956698 5.5104333540991556298e-16 -3.1415926535897926719 -> xyz=0.27499999999999591438 5.5511151231257827021e-16 0.02999999999999993644 rpy=-1.5707963267948945596 1.109557078629070938e-15 3.141592653589793116
- joint l4_cl2_1_frame: origin xyz=5.5511151231257827021e-17 0 -0.0094999999999996198596 rpy=-1.57079632679489678 -1.5707963267948958919 0 -> xyz=1.1102230246251565404e-16 1.1102230246251565404e-16 -0.0094999999999998419042 rpy=-1.57079632679489678 -1.570796326794896336 0
- joint l4_cl2_2_frame: origin xyz=-0.012999999999999678479 0.3840000000000000635 0.019999999999999795719 rpy=1.570796326794896558 -4.8590027552132278873e-16 -2.6823769382526587703e-16 -> xyz=-0.012999999999999789502 0.38399999999999984146 0.020000000000000017764 rpy=1.5707963267948981123 5.6418899027106805647e-15 -8.2747863375710439487e-17
- joint l4_cl3_1_frame: origin xyz=-2.2204460492503130808e-16 -2.2204460492503130808e-16 -0.0094999999999996198596 rpy=1.570796326794896558 1.5707963267948952257 0 -> xyz=-5.5511151231257827021e-16 -4.4408920985006261617e-16 -0.0094999999999998419042 rpy=1.57079632679489678 1.570796326794896336 0
- joint l4_cl3_2_frame: origin xyz=0 -0.50500000000000011546 0.020000000000000295319 rpy=-1.570796326794896558 1.0095225613817616779e-15 -3.141592653589793116 -> xyz=0 -0.50500000000000011546 0.020000000000000239808 rpy=-1.5707963267948983344 4.250158188698657927e-15 3.141592653589793116
- joint l4_cl4_1_frame: origin xyz=-1.1102230246251565404e-16 0.59000000000000030198 0.01999999999999985123 rpy=1.57079632679489678 -7.2679738829527707955e-16 3.1415926535897917837 -> xyz=-1.1102230246251565404e-16 0.59000000000000030198 0.020000000000000239808 rpy=1.570796326794896558 -2.1172771087553852848e-17 3.141592653589793116
- joint l4_cl4_2_frame: origin xyz=-0.45000000000000039968 0 -0.020000000000000073275 rpy=-1.570796326794896558 1.2508912073766756774e-16 -3.141592653589793116 -> xyz=-0.45000000000000117684 1.1102230246251565404e-16 -0.020000000000001016964 rpy=-1.570796326794896558 -1.3365231167518776006e-16 -3.141592653589793116
- joint l4_r1: origin xyz=-0.18999999999999961364 -0.96499999999999985789 1.0755285551056070865e-16 rpy=3.1415926535897908956 1.9044041489550536811e-24 0.28196247148250824788 -> xyz=-0.18999999999999969691 -0.96500000000000030198 1.0755285551056218776e-16 rpy=3.1415926535897922278 -2.294689447613700712e-16 0.14573630623988689803
- joint l4_r2: origin xyz=0.5 -1.0249999999999999112 0.030000000000000099504 rpy=-3.1415926535897926719 7.8766131130756764154e-16 2.2857888156166228377 -> xyz=0.49999999999999933387 -1.0249999999999996891 0.030000000000000116851 rpy=3.1415926535897926719 -6.4212163323135518491e-16 2.6683037279205028547
- joint l4_r3: origin xyz=0.12500000000000732747 -0.019999999999993856026 -0.039999999999999896749 rpy=-1.5707963267948958919 0.35430516897449731983 1.1506556893667557454e-14 -> xyz=0.125 -0.020000000000000239808 -0.040000000000000021649 rpy=-1.570796326794896558 0.4666163750680140665 -1.6377357379776283407e-14
- joint l4_r4: origin xyz=1.1102230246251565404e-15 0.48999999999999860334 2.0539125955565395998e-15 rpy=3.1415926535897895633 4.8455040699935128072e-15 -0.35430516897449099156 -> xyz=-4.2188474935755948536e-15 0.48999999999999549471 -2.4424906541753443889e-15 rpy=3.1415926535897908956 -2.3344824489569353479e-14 -0.4152831526151581909
- joint l4_r5: origin xyz=-0.75 3.3306690738754696213e-16 -0.040000000000000035527 rpy=-6.4405352938840367248e-15 8.4157945655509966573e-15 -3.141592653589793116 -> xyz=-0.74999999999999966693 0 -0.039999999999999813483 rpy=-4.1114399506133858885e-17 -3.1816225832927581697e-17 2.876806338808024055
- joint l4_r6: origin xyz=-0.40999999999999836575 1.4988010832439613296e-15 -0.094999999999999917843 rpy=1.5707963267949027752 0.65724109672369257495 3.5697696165855604194e-15 -> xyz=-0.40999999999999747757 -8.8817841970012523234e-16 -0.094999999999998280265 rpy=1.5707963267948974462 0.67749592276418513226 -2.3346654462577296161e-15
- joint l4_r7: origin xyz=-0.12500000000000133227 -0.019999999999999684697 -0.03999999999999995226 rpy=-1.5707963267949001107 0.67784852797314421036 -1.4595506346581353191e-14 -> xyz=-0.125 -0.020000000000000128786 -0.039999999999999993894 rpy=-1.57079632679489678 0.79176818239134705291 3.9765294598519190235e-15
- joint l4_r8: origin xyz=0 0.3925000000000002931 0.019999999999999573674 rpy=3.5707879082592744506e-15 2.3225679053517195645e-14 -3.127565063384278865 -> xyz=-1.1102230246251565404e-16 0.39250000000000051514 0.019999999999999684697 rpy=-6.1759297529534193009e-16 2.3607132528423478458e-16 -3.0336414428136180277
- joint leg_1_frame: origin xyz=0.004999999999999671374 -1.0075000000000000622 0.020000000000000239808 rpy=-1.570796326794896558 -3.7290365520547414402e-16 -1.4139732311379854492e-28 -> xyz=0.0050000000000001154632 -1.0075000000000002842 0.019999999999999972661 rpy=-1.570796326794896558 -1.6917805583653369258e-16 -2.2741465533138622391e-17
- joint leg_2_frame: origin xyz=0.0049999999999998934186 -1.0074999999999998401 0.020000000000000184297 rpy=-1.570796326794896558 2.1015511443037622533e-16 -5.1910748321200000537e-18 -> xyz=0.0050000000000001154632 -1.0074999999999998401 0.020000000000000073275 rpy=-1.570796326794896558 5.1401146879175467997e-16 -6.56223101404631036e-17
- joint leg_3_frame: origin xyz=0.0049999999999998934186 -1.0074999999999998401 0.020000000000000017764 rpy=-1.570796326794896558 -1.0354129802097694568e-16 -6.2450045135172953869e-16 -> xyz=0.0049999999999998934186 -1.0075000000000000622 0.019999999999999962252 rpy=-1.57079632679489678 3.302719205854473423e-16 9.2428687743045562232e-17
- joint leg_4_frame: origin xyz=0.0050000000000001154632 -1.0075000000000000622 0.020000000000000073275 rpy=-1.570796326794896558 -8.3307679057966979047e-16 8.3266726846905118526e-17 -> xyz=0.0050000000000001154632 -1.0075000000000000622 0.020000000000000017764 rpy=-1.57079632679489678 8.44481009585997054e-17 4.062073120193065484e-17
