Commit message: Adjusting limits in the quadruped model

File: models/quadruped/robot.urdf (robot description, URDF)
Before this commit: robot onshape, 18 links, 17 joints
Joints:
- joint leg1_a: limit lower=-1.570796326794896558 upper=1.570796326794896558 effort=1 velocity=20 -> lower=-1.570796326794896558 upper=1.570796326794896558 effort=1 velocity=12
- joint leg1_b: limit lower=-1.570796326794896558 upper=1.570796326794896558 effort=1 velocity=20 -> lower=-1.570796326794896558 upper=1.570796326794896558 effort=1 velocity=12
- joint leg1_c: limit effort=1 velocity=20 -> lower=0.0 upper=3.1415926 effort=1 velocity=12
- joint leg2_a: limit lower=-1.570796326794896558 upper=1.570796326794896558 effort=1 velocity=20 -> lower=-1.570796326794896558 upper=1.570796326794896558 effort=1 velocity=12
- joint leg2_b: limit lower=-1.570796326794896558 upper=1.570796326794896558 effort=1 velocity=20 -> lower=-1.570796326794896558 upper=1.570796326794896558 effort=1 velocity=12
- joint leg2_c: limit effort=1 velocity=20 -> lower=0.0 upper=3.1415926 effort=1 velocity=12
- joint leg3_a: limit lower=-1.570796326794896558 upper=1.570796326794896558 effort=1 velocity=20 -> lower=-1.570796326794896558 upper=1.570796326794896558 effort=1 velocity=12
- joint leg3_b: limit lower=-1.570796326794896558 upper=1.570796326794896558 effort=1 velocity=20 -> lower=-1.570796326794896558 upper=1.570796326794896558 effort=1 velocity=12
- joint leg3_c: limit effort=1 velocity=20 -> lower=0.0 upper=3.1415926 effort=1 velocity=12
- joint leg4_a: limit lower=-1.570796326794896558 upper=1.570796326794896558 effort=1 velocity=20 -> lower=-1.570796326794896558 upper=1.570796326794896558 effort=1 velocity=12
- joint leg4_b: limit lower=-1.570796326794896558 upper=1.570796326794896558 effort=1 velocity=20 -> lower=-1.570796326794896558 upper=1.570796326794896558 effort=1 velocity=12
- joint leg4_c: limit effort=1 velocity=20 -> lower=0.0 upper=3.1415926 effort=1 velocity=12
