Commit message: Differential model

File: models/differential/robot.urdf (robot description, URDF)
Before this commit: robot onshape, 5 links, 4 joints
Links:
- added link effector, mass 1e-9
- link shaft1: mass 0.024130399999999996297 -> 0.0086799999999999984807
- link shaft2: mass 0.046198276629261847415 -> 0.028491984468144111731
Joints:
- added joint effector_frame: type fixed, parent shaft2, child effector, origin xyz=0.049667853818713914027 -0.068361936024683156443 -0.02749999999999998973 rpy=0.942477796076938934 1.570796326794896558 0, axis 0 0 0
- joint alpha: origin xyz=-4.3335586649446777637e-18 1.9137705312060885725e-18 0.004999999999999997502 rpy=0 -0 0.31923972210080497902 -> xyz=0 1.3777276490407720037e-18 0.004999999999999997502 rpy=0 -0 1.570796326794896558
- joint beta: origin xyz=-4.725960828366940336e-18 -0.0075000000000000023245 0.01999999999999997613 rpy=-1.570796326794896558 -0 0 -> xyz=-1.3777276490407427296e-18 -0.0074999999999999997224 0.019999999999999996947 rpy=-1.570796326794896558 -0.62831853071796783805 -2.0584666929331748659e-16
- joint upper: origin xyz=0 1.3777276490407725815e-18 0.044999999999999998335 rpy=0 -0 0 -> xyz=3.4694469519536141888e-18 1.3777276490407700778e-18 0.044999999999999998335 rpy=3.4000580129145483145e-16 -9.788590809453151338e-17 -2.8085211743323700543e-18
