Commit message: Updating SPM orientation & zero

File: models/spm/robot.urdf (robot description, URDF)
Before this commit: robot spm, 13 links, 12 joints
Joints:
- joint closing_m1_p2_1_frame: origin xyz=0.0279738 2.02616e-15 -0.0497913 rpy=-3.14159 -1.31812 -1.44912e-15 -> xyz=0.0279738 2.02616e-15 -0.0497913 rpy=-3.14159 -1.31812 -1.62357e-15
- joint closing_m1_p2_2_frame: origin xyz=-0.0258211 0.0107611 0.0216684 rpy=-1.82348 4.07601e-14 1.17593 -> xyz=-0.0279738 -5.82867e-16 0.0216684 rpy=-1.82348 -7.45088e-15 1.5708
- joint closing_m3_p2_1_frame: origin xyz=0.0227371 -0.0162959 -0.0497913 rpy=-3.14159 -1.31812 -0.621854 -> xyz=0.0279738 1.6237e-15 -0.0497913 rpy=-3.14159 -1.31812 -1.81564e-14
- joint closing_m3_p2_2_frame: origin xyz=-0.0157079 -0.0231472 0.0216684 rpy=1.95839 -0.848062 -0.893349 -> xyz=-0.00559476 -0.0274086 0.0216684 rpy=1.95839 -0.848062 -0.49848
- joint effector_frame: origin xyz=-0.0227072 -0.00677243 0.0051956 rpy=2.42787 -0.361367 -1.66854 -> xyz=-0.0183545 -0.0149864 0.0051956 rpy=2.42787 -0.361367 -1.27367
- joint m1: origin xyz=-0.0256569 0.044439 0.0612132 rpy=2.39619 0.275486 -2.33141 -> xyz=-0.0513137 2.95076e-15 0.0612132 rpy=2.35619 -9.97813e-15 -1.5708
- joint m2: origin xyz=-0.0256569 -0.044439 0.0612132 rpy=-2.35619 1.99341e-16 2.61799 -> xyz=0.0256569 -0.044439 0.0612132 rpy=-2.35619 1.99341e-16 -2.61799
- joint m2_p1: origin xyz=-0.0117802 0.0394975 -0.0619264 rpy=1.31313 0.19488 -2.90273 -> xyz=-0.0260678 0.0319264 -0.0619264 rpy=1.31313 0.19488 -2.50786
- joint m2_p2: origin xyz=0.0227371 -0.0162959 -0.0497913 rpy=-1.13637e-14 -1.31812 -0.621854 -> xyz=0.0279738 2.2829e-15 -0.0497913 rpy=-3.36345e-14 -1.31812 6.54005e-15
- joint m3: origin xyz=0.0513137 2.63504e-15 0.0612132 rpy=-2.35619 3.18634e-14 -1.5708 -> xyz=0.0256569 0.044439 0.0612132 rpy=-2.35619 3.18634e-14 -0.523599
- joint m3_p1: origin xyz=-0.0117802 0.0394975 -0.0619264 rpy=1.20784 0.789565 -3.11514 -> xyz=-0.0260678 0.0319264 -0.0619264 rpy=1.31313 0.19488 -2.50786
